File: kicad/pcb/pcb.kicad_pcb (KiCad board)
At the start: 2 copper layers, 89.8 x 108 mm, 91 parts, among them J1 Conn_01x04, SW1 SW_SPST, SW10 SW_SPST, SW11 SW_SPST, SW12 SW_SPST, SW13 SW_SPST, SW14 SW_SPST, SW15 SW_SPST, SW16 SW_SPST, SW17 RotaryEncoder_Switch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

Commit message: add gerbers, BOM, firmware, schematic, assets, license
Parts:
- moved D14 1.10 mm to (98.9, 115.5)
- moved C11 0.99 mm to (160.6, 147.7)
Routing:
- net Net-(D14-A): track 7.68 -> 6.47 mm
- net R4: track 100.4 -> 99.8 mm
Other:
- board text added: "Codemate-v2"
- board text added: "TX"
- board text added: "from aryan-git-byte"

Commit message: complete
Parts:
- moved C11 0.91 mm to (161.3, 147.2)
Changed lines of the file:
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@@
 	(footprint "Capacitor_SMD:C_0603_1608Metric"
 		(layer "F.Cu")
-		(at 160.55 147.675 -90)
+		(at 161.35 147.25 -90)
 		(descr "Capacitor SMD 0603 (1608 Metric), square (rectangular) end terminal, IPC-7351 nominal, (Body size source: IPC-SM-782 page 76, https://www.pcb-3d.com/wordpress/wp-content/uploads/ipc-sm-782a_amendment_1_and_2.pdf), generated with kicad-footprint-generator")
 		(tags "capacitor")
