File: kicad/pcb/pcb.kicad_sch (KiCad schematic)
At the start: 88 parts, among them J1 Conn_01x04, SW1 SW_SPST, SW10 SW_SPST, SW11 SW_SPST, SW12 SW_SPST, SW13 SW_SPST, SW14 SW_SPST, SW15 SW_SPST, SW16 SW_SPST, SW17 RotaryEncoder_Switch, SW18 RotaryEncoder_Switch, SW2 SW_SPST, SW3 SW_SPST, SW4 SW_SPST, SW5 SW_SPST, SW6 SW_SPST, SW7 SW_SPST, SW8 SW_SPST, SW9 SW_SPST, U1 ESP32-S3-ZERO, U2 PCF8574AP

Commit message: add gerbers, BOM, firmware, schematic, assets, license
Connections:
- no-connect marks 0 -> 1
Other:
- moved on the sheet: C1, C10, C11, C12, C13, C14, C15, C16, C17, C18, C19, C2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

Commit message: complete
Parts:
- renumbered C20 to C1, C23 to C10, C1 to C11, C2 to C12, C3 to C13, C4 to C14, C5 to C15, C6 to C16, C7 to C17, C8 to C18, C15 to C19, C17 to C2, C10 to C20, C9 to C21, C16 to C22, C12 to C23, C11 to C24, C21 to C25, C13 to C3, C14 to C4, C19 to C5, C18 to C6, C22 to C7, C25 to C8, C24 to C9, D32 to D1, D29 to D10, D30 to D11, D22 to D12, D21 to D13, D20 to D14, D27 to D15, D26 to D16, D25 to D17, D24 to D18, D23 to D19, D33 to D2, D37 to D20, D38 to D21, D39 to D22, D40 to D23, D41 to D24, D31 to D25, D1 to D26, D2 to D27, D3 to D28, D4 to D29, D34 to D3, D5 to D30, D6 to D31, D7 to D32, D8 to D33, D9 to D34, D10 to D35, D11 to D36, D12 to D37, D13 to D38, D14 to D39, D35 to D4, D15 to D40, D16 to D41, D36 to D5, D28 to D6, D19 to D7, D18 to D8, D17 to D9, SW17 to SW10, SW9 to SW11, SW10 to SW12, SW11 to SW13, SW12 to SW14, SW13 to SW15, SW14 to SW16, SW15 to SW17, SW16 to SW18, SW18 to SW5, SW5 to SW6, SW6 to SW7, SW7 to SW8, SW8 to SW9
Connections:
- no-connect marks 1 -> 3
